File: kicad/03_llc.kicad_sch (KiCad schematic)
At the start: 64 parts, among them J301 48V OUT, Q301 IPP60R099C7, Q302 IPP60R099C7, Q310 BSC070N10NS3, Q311 BSC070N10NS3, Q312 BSC070N10NS3, Q313 BSC070N10NS3, T301 EE35 50:(12+12), U301 L6599D, U302 UCC24610D, U303 UCC24610D, U304 INA181A2, U305 TL431BDBZR, U306 PC817

Commit message: Этап 3.1: уточнения по даташитам (L6599 RFmin/RFmax/Css, замена UCC24610→UCC24624)
- websearch-верификация: L6599 RFmin — 2В источник, ветви RFmin/RFmax/Css-Rss,
  полярность ОС подтверждена (ток↑→частота↑→Vout↓); пин 2/13 N.C.
- UCC24610 не применим: VD макс 50В против ~96В на стоке SR при 48В выходе;
  SYNC к GND удерживал бы GATE выкл.
- Добавлен символ psu48_lib:UCC24624 (SOIC-8, VT до 230В, 2 канала)
- Схема 03: 1×UCC24624 вместо 2×UCC24610; R328 4.7k RFmax; R308 мягкий старт;
  удалены U303/R314/R315/C314 и старая ветка LLC_DLY
- verify 433 вывода OK, ERC 0/0, qa чисто
- docs/DESIGN.md актуализирован (UCC24624)
Parts:
- removed C303, C314: 100nF, Capacitor_SMD:C_0805_2012Metric, symbol Device:C
- removed R314, R315: 10k, Resistor_SMD:R_0805_2012Metric, symbol Device:R
- removed U303: UCC24610D, Package_SO:SOIC-8_3.9x4.9mm_P1.27mm, symbol Regulator_Controller:UCC24610D
- added C316: 2.2uF, Capacitor_SMD:C_0805_2012Metric, symbol Device:C
- added R328: 4.7k, Resistor_SMD:R_0805_2012Metric, symbol Device:R
- U302: value UCC24610D -> UCC24624; symbol Regulator_Controller:UCC24610D -> psu48_lib:UCC24624
Connections:
- net +15VS: now also U302.7 (VDD); no longer U302.2 (EN/TOFF), U302.4 (VCC)
- net GND: no longer R308.2
- net GND48: now also U302.2 (PGND), U302.5 (VSS), C316.2; no longer U302.1 (SYNC), U302.6 (GND), U302.7 (VS)
- net G_SR1: now also U302.1 (VG1); no longer U302.5 (GATE)
- net G_SR2: now also U302.8 (VG2)
- net LLC_CSS: now also R308.1
- net LLC_FB: now also R308.2, R328.1; no longer U306.4
- net SEC_A: now also U302.4 (VD1); no longer U302.8 (VD)
- net SEC_B: now also U302.6 (VD2)
- net LLC_DLY: no longer names the net of U301.2 (DELAY)
- net LLC_DLY: no longer R308.1
- net SR_TON1 renamed SR_REG
- net SR_REG: now also C316.1
- new net LLC_OPTO: R328.2, U306.4
- no-connect marks 1 -> 2
Other:
- moved on the sheet: C304, C305, C306, C313, C320, C321, C322, C323, C324, C325, C326, C327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

Commit message: Этап 4: генерация PCB (pcbgen: 167 корпусов + 4 отверстия), размещение, DRC без ошибок; правки схемы (SEC_A->AUX_SEC, LED_A->STATUS_LED)
Other:
- moved on the sheet: C310, C311, C313, C316, C320, C321, C322, C323, C324, C325, Q311, Q312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
