File: kicad/04_aux.kicad_sch (KiCad schematic)
At the start: 25 parts, among them J401 FAN 12V, T401 EE16 flyback, U401 TNY290PG, U402 PC817, U403 TL431BDBZR, U404 L7812CV

Commit message: Этап 4: генерация PCB (pcbgen: 167 корпусов + 4 отверстия), размещение, DRC без ошибок; правки схемы (SEC_A->AUX_SEC, LED_A->STATUS_LED)
Connections:
- net SEC_A renamed AUX_SEC
Other:
- moved on the sheet: C401, C402, C405, C406, C408, C409, C410, D402, J401, R401, R402, R403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
