File: kicad/psu48.kicad_pcb (KiCad board)
At the start: 2 copper layers, 280 x 90 mm, 171 parts, among them J101 AC IN 220V, J301 48V OUT, J401 FAN 12V, J501 PG ON_OFF GND, K101 G2RL-2 DC12, Q101 MMBT3904, Q201 IPP60R099C7, Q301 IPP60R099C7, Q302 IPP60R099C7, Q310 BSC070N10NS3, Q311 BSC070N10NS3, Q312 BSC070N10NS3, Q313 BSC070N10NS3, T301 EE35 50:(12+12), T401 EE16 flyback, U201 UC3854GN, U202 LM393DR, U301 L6599D, U302 UCC24624, U304 INA181A2, U305 TL431BDBZR, U306 PC817, U401 TNY290PG, U402 PC817, U403 TL431BDBZR, U404 L7812CV, U501 LM393DR, U502 LM393DR, U503 TL431BDBZR, U504 PC817, U505 PC817

Commit message: Этап 5 (черновик): автотрассировка router.py — валидный вывод для KiCad 10 ((net <code>)+uuid), 712 треков/595 виа; диагноз DRC (co-located vias, асимметричный зазор ширин); журнал
Routing:
- net 04_aux/AUX_FB: track 0.00 -> 696.1 mm, vias 0 -> 27
- net GND: track 0.00 -> 394.7 mm, vias 0 -> 35
- net 03_llc/PRI_B: track 0.00 -> 355.5 mm, vias 0 -> 18
- net VBUS400: track 0.00 -> 324.9 mm, vias 0 -> 10
- net 05_ctrl/PG_SENSE: track 0.00 -> 318.7 mm, vias 0 -> 28
- net 03_llc/LLC_CSS: track 0.00 -> 297.0 mm, vias 0 -> 28
- net 04_aux/AUX_CL: track 0.00 -> 292.1 mm, vias 0 -> 9
- net GND48: track 0.00 -> 278.9 mm, vias 0 -> 69
- net 02_pfc/PFC_VS: track 0.00 -> 271.2 mm, vias 0 -> 7
- net 03_llc/HS: track 0.00 -> 266.9 mm, vias 0 -> 3
- net 03_llc/VBOOT: track 0.00 -> 241.9 mm, vias 0 -> 11
- net +12V: track 0.00 -> 233.6 mm, vias 0 -> 8
- net 02_pfc/PFC_SS: track 0.00 -> 231.4 mm, vias 0 -> 10
- net ISENSE_48: track 0.00 -> 231.4 mm, vias 0 -> 16
- net +15V: track 0.00 -> 229.1 mm, vias 0 -> 13
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